File: hardware/Uzebox F6/Uzebox Game Console F6.sch (EAGLE design)
At the start: 81 parts, among them CON1 USBSERIALSMD, IC1 MCP1700, IC2 7805T, U5 DC IN, U6 23LC1024, X1 MINI-DIN-9

Commit message: Update layout for better silkscreen
Parts:
- X1: value MINI-DIN-9 -> A/V
Changed lines of the file:
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@@
 <part name="C17" library="adafruit" deviceset="CPOL-US" device="E2-4" value="1uF"/>
 <part name="P+9" library="supply1" deviceset="+5V" device=""/>
-<part name="X1" library="Thorsten_connectors" deviceset="MINI-DIN-9" device=""/>
+<part name="X1" library="Thorsten_connectors" deviceset="MINI-DIN-9" device="" value="A/V"/>
 <part name="P+10" library="supply1" deviceset="+5V" device=""/>
 <part name="R4" library="resistor" deviceset="R-US_" device="0207/10" value="180"/>
